File: board/vgascart.kicad_pcb (KiCad board)
At the start: 2 copper layers, 46 x 59 mm, 9 parts, among them J4 SCART-F, J5 Conn_Coaxial, J6 DB15_Female_HighDensity, J7 AudioJack3, J8 Comp/Sync

Commit message: Board cleanup, README
Parts:
- J8: value Comp/Sync -> Comp Sync
Other:
- board text added: "© 2022 Simon Kowalewski"
- board text removed: "https://www.youtube.com /c/SimonKowalewski"
